File: MS_Picosensor_PCB.kicad_pcb (KiCad board)
At the start: 2 copper layers, 78.4 x 78 mm, 24 parts, among them J1 Conn_01x20_Socket, J2 Conn_01x20_Socket, J3 Conn_01x06_Socket, J4 Conn_01x02_Socket, J5 Conn_01x02, J6 Screw_Terminal_01x03, J7 SM04B-SRSS-TB, SW1 SW_MEC_5E, SW2 SW_MEC_5E, SW3 SW_DIP_x01

Commit message: 3v3 output
Parts:
- removed R2, R3: 1K, Resistor_THT:R_Axial_DIN0207_L6.3mm_D2.5mm_P10.16mm_Horizontal
- R4, R5: value 330 -> 220
Connections:
- J2 pad 4: +3.3V -> Net-(J2-Pin_4)
- J2 pad 5: Net-(J2-Pin_5) -> +3.3V
Routing:
- net +3.3V: track 155.2 -> 144.4 mm
- net /RButton: track 49.4 -> 41.3 mm
